File: TSL2561_v0.1.brd (EAGLE design)
At the start: 17.8 x 17 mm, 10 parts, among them U1 TSL2561

Commit message: Add files via upload
Routing:
- net INT: track 6.82 -> 6.08 mm
Changed lines of the file:
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@@
 <contactref element="U1" pad="INT"/>
 <contactref element="JP1" pad="3"/>
-<wire x1="8.89" y1="6.858" x2="8.89" y2="8.09" width="0.254" layer="1"/>
-<wire x1="7.62" y1="6.858" x2="8.89" y2="6.858" width="0.254" layer="1"/>
-<wire x1="7.62" y1="2.54" x2="7.62" y2="6.858" width="0.254" layer="1"/>
+<wire x1="8.89" y1="5.334" x2="8.89" y2="8.09" width="0.254" layer="1"/>
+<wire x1="7.62" y1="4.064" x2="8.89" y2="5.334" width="0.254" layer="1"/>
+<wire x1="7.62" y1="2.54" x2="7.62" y2="4.064" width="0.254" layer="1"/>
 </signal>
 <signal name="ADDR">
